File: PCB_LEDCube/PCB_LEDCube.kicad_pcb (KiCad board)
At the start: 2 copper layers, 72 parts, among them J1 Source, J2 Batt, Q1 2N2219, Q10 2N2219, Q2 2N2219, Q3 2N2219, Q4 2N2219, Q5 2N2219, Q6 2N2219, Q7 2N2219, Q8 2N2219, Q9 2N2219, U1 L7805, U2 MCP73931, U3 WemosESP32, U4 74HC595, U5 74HC595

Commit message: PCB TH hand
Parts:
- removed C1, C5: 10uf, Capacitor_SMD:C_1206_3216Metric_Pad1.42x1.75mm_HandSolder
- removed D2: ON, LED_SMD:LED_1206_3216Metric_Pad1.42x1.75mm_HandSolder
- removed D3: Charging, LED_SMD:LED_1206_3216Metric_Pad1.42x1.75mm_HandSolder
- removed D4: D_Schottky, Diode_THT:D_A-405_P7.62mm_Horizontal
- removed J2: Batt, Connector_PinHeader_2.54mm:PinHeader_1x02_P2.54mm_Vertical
- removed JP1: SJ1, Jumper:SolderJumper-2_P1.3mm_Open_RoundedPad1.0x1.5mm
- removed R1, R2: 470R, Resistor_SMD:R_1206_3216Metric_Pad1.42x1.75mm_HandSolder
- removed R3: 10k, Resistor_SMD:R_1206_3216Metric_Pad1.42x1.75mm_HandSolder
- removed R4: 2k, Resistor_SMD:R_1206_3216Metric_Pad1.42x1.75mm_HandSolder
- removed U2: MCP73931, Package_TO_SOT_SMD:SOT-23-5
- C2, C3: footprint Capacitor_SMD:C_1206_3216Metric_Pad1.42x1.75mm_HandSolder -> Capacitor_THT:C_Disc_D5.0mm_W2.5mm_P5.00mm
- R10, R11, R12, R13, R14, R15, R16, R17, R18, R19, R20, R21, R22, R23, R24, R25, R26, R27, R28, R29, R30, R5, R6, R7, R8, R9: footprint Resistor_SMD:R_1206_3216Metric_Pad1.42x1.75mm_HandSolder -> Resistor_THT:R_Axial_DIN0207_L6.3mm_D2.5mm_P7.62mm_Horizontal
- moved R20 176.2 mm to (47.5, 173.0), turned to 180 degrees
- moved C2 169.8 mm to (18.6, 80.7)
- moved C3 161.0 mm to (28.4, 94.3), turned to 180 degrees
- moved R26 144.6 mm to (76.8, 169.5), turned to 180 degrees
- moved J1 134.1 mm to (20.7, 49.2), turned to 270 degrees
- moved Q7 133.7 mm to (47.2, 145.9)
- moved Q10 130.3 mm to (75.5, 164.3)
- moved R19 130.1 mm to (48.0, 152.2), turned to 180 degrees
- moved R8 121.0 mm to (81.2, 25.7)
- moved R9 114.5 mm to (79.8, 44.6)
- moved Q5 112.5 mm to (84.8, 38.5)
- moved Q8 112.4 mm to (46.1, 167.8)
- moved Q4 112.0 mm to (85.9, 18.5)
- moved R6 107.5 mm to (80.0, 100.1)
- moved D1 98.3 mm to (15.6, 71.0)
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Connections:
- C2 pad 1: +12V -> Net-(C2-Pad1)
- C2 pad 2: +12V -> GND
- C3 pad 2: +12V -> GND
- D1 pad 1: +12V -> Net-(C2-Pad1)
- J1 pad 1: +12V -> GND
- Q10 pad 1: +12V -> GND
- Q7 pad 1: +12V -> GND
- Q8 pad 1: +12V -> GND
- Q9 pad 1: +12V -> GND
- U1 pad 1: +12V -> Net-(C2-Pad1)
- U1 pad 2: +12V -> GND
- U3 pad 10: +12V -> GND
- U3 pad 24: +12V -> GND
- U3 pad 25: +12V -> GND
- U3 pad 40: +12V -> GND
- U4 pad 13: +12V -> GND
- U4 pad 8: +12V -> GND
- U5 pad 13: +12V -> GND
- U5 pad 8: +12V -> GND

Commit message: pcb desing
Parts:
- added J2: GND, Connector_PinHeader_2.54mm:PinHeader_1x03_P2.54mm_Vertical, F.Cu at (158.0, 115.0)
- moved J1 175.3 mm to (167.6, 144.8), turned to 180 degrees
- moved D1 154.2 mm to (155.0, 137.0)
- moved C2 149.1 mm to (155.0, 141.0), turned to 270 degrees
- moved U1 140.3 mm to (150.0, 142.0), turned to 180 degrees
- moved R19 134.9 mm to (180.0, 124.5)
- moved Q7 134.4 mm to (179.0, 119.4)
- moved Q8 128.4 mm to (165.0, 119.4)
- moved R20 128.1 mm to (166.0, 124.5)
- moved C3 121.0 mm to (140.0, 141.0), turned to 270 degrees
- moved Q9 120.4 mm to (193.0, 119.4)
- moved R25 120.2 mm to (194.0, 124.5)
- moved U3 105.3 mm to (121.9, 129.5)
- moved D18 104.6 mm to (152.4, 25.3)
- moved R28 102.2 mm to (144.8, 25.3)
- moved D5 89.9 mm to (228.6, 101.6)
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Connections:
- D10 pad 1: /GND2 -> /GND4
- D11 pad 1: /GND2 -> /GND4
- D12 pad 1: /GND2 -> /GND4
- D13 pad 1: /GND3 -> /GND4
- D14 pad 1: /GND3 -> /GND4
- D15 pad 1: /GND3 -> /GND4
- D16 pad 1: /GND3 -> /GND4
- D5 pad 1: /GND1 -> /GND4
- D6 pad 1: /GND1 -> /GND4
- D7 pad 1: /GND1 -> /GND4
- D8 pad 1: /GND1 -> /GND4
- D9 pad 1: /GND2 -> /GND4
- Q1 pad 2: /IO18 -> /IO23
- Q2 pad 2: /IO16 -> /IO18
- Q3 pad 2: /IO17 -> /IO19
- Q4 pad 2: /IO21 -> /IO35
- Q5 pad 2: /IO22 -> /IO34
- Q6 pad 2: /IO23 -> /IO33
- R26 pad 2: /IO5 -> /IO32
Routing:
- net /GND4: track 0.00 -> 476.8 mm
- net GND: track 0.00 -> 433.3 mm, vias 0 -> 3
- net +5V: track 0.00 -> 204.5 mm
- net /IO34: track 0.00 -> 142.4 mm
- net /IO33: track 0.00 -> 109.6 mm
- net /F5: track 0.00 -> 95.0 mm
- net /F13: track 0.00 -> 93.5 mm
- net /IO35: track 0.00 -> 93.3 mm
- net /F12: track 0.00 -> 87.4 mm
- net /F4: track 0.00 -> 87.4 mm
- net /F6: track 0.00 -> 67.1 mm
- net /F14: track 0.00 -> 66.8 mm
- net /IO18: track 0.00 -> 63.6 mm
- net /F3: track 0.00 -> 59.5 mm
- net /F11: track 0.00 -> 59.5 mm
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Other:
- board outline added: 142.2 x 129.5 mm
- net class Default: trace_width 0.25 -> 1
- board text added: "3R"
