File: PCB_LEDCube/PCB_LEDCube.sch (KiCad schematic (older format))
At the start: 20 parts

Commit message: Add footprints
Parts:
- removed C? (x2): 10uf, Capacitor_SMD:C_1206_3216Metric_Pad1.42x1.75mm_HandSolder, symbol Device:C
- removed U?: LF33_TO220, Package_TO_SOT_THT:TO-220-3_Vertical, symbol Regulator_Linear:LF33_TO220
- added D10, D11, D12, D13, D14, D15, D16, D17, D18, D19, D20, D5, D6, D7, D8, D9: LED, LED_THT:LED_D5.0mm, symbol Device:LED
- added Q1, Q10, Q2, Q3, Q4, Q5, Q6, Q7, Q8, Q9: 2N2219, Package_TO_SOT_THT:TO-92L_Inline, symbol Transistor_BJT:2N2219
- added R10, R11, R12, R13, R14, R15, R16, R17, R18, R19, R20, R21, R22, R23, R24, R25, R26, R27, R28, R29, R30, R5, R6, R7, R8, R9: 220, Resistor_SMD:R_1206_3216Metric_Pad1.42x1.75mm_HandSolder, symbol Device:R
- added U3: WemosESP32, ESP32_Wemos:Wemos_ESP32, symbol IC:WemosESP32
- added U4, U5: 74HC595, Package_DIP:DIP-16_W10.16mm_LongPads, symbol 74xx:74HC595
- D1, D4: renamed from D?; footprint (none) -> Diode_THT:D_A-405_P7.62mm_Horizontal
- U1: renamed from U?; footprint (none) -> Package_TO_SOT_THT:TO-220-3_Vertical
- U2: renamed from U?; symbol Regulator:MCP73931 -> PCB_LEDCube-rescue:MCP73931-Regulator
- gave numbers to parts that had none: 13
Connections:
- net labels added: +12V, F1, F10, F11, F12, F13, F14, F15, F16, F2, F3, F4, F5, F6, F7, F8, F9, GND1, GND2, GND3, GND4, IO0, IO16, IO17, IO18, IO19, IO2, IO21, IO22, IO23, IO25, IO26, IO27, IO32, IO33, IO34, IO35, IO4, IO5, RCLK1, RCLK2, SER1, SER2, SRCLK1, SRCLK2
- net labels removed: +3.3V
- wire segments 73 -> 130
- no-connect marks 0 -> 19
Other:
- note removed: "Regulator 3.3V"
- moved on the sheet: C2, C3, D1, D4, J1, U1

Commit message: PCB TH hand
Parts:
- removed C1, C5: 10uf, Capacitor_SMD:C_1206_3216Metric_Pad1.42x1.75mm_HandSolder, symbol Device:C
- removed D2: ON, LED_SMD:LED_1206_3216Metric_Pad1.42x1.75mm_HandSolder, symbol Device:LED
- removed D3: Charging, LED_SMD:LED_1206_3216Metric_Pad1.42x1.75mm_HandSolder, symbol Device:LED
- removed D4: D_Schottky, Diode_THT:D_A-405_P7.62mm_Horizontal, symbol Device:D_Schottky
- removed J2: Batt, Connector_PinHeader_2.54mm:PinHeader_1x02_P2.54mm_Vertical, symbol Connector:Conn_01x02_Female
- removed JP1: SJ1, Jumper:SolderJumper-2_P1.3mm_Open_RoundedPad1.0x1.5mm, symbol Device:Jumper_NO_Small
- removed R1, R2: 470R, Resistor_SMD:R_1206_3216Metric_Pad1.42x1.75mm_HandSolder, symbol Device:R
- removed R3: 10k, Resistor_SMD:R_1206_3216Metric_Pad1.42x1.75mm_HandSolder, symbol Device:R
- removed R4: 2k, Resistor_SMD:R_1206_3216Metric_Pad1.42x1.75mm_HandSolder, symbol Device:R
- removed U2: MCP73931, Package_TO_SOT_SMD:SOT-23-5, symbol PCB_LEDCube-rescue:MCP73931-Regulator
- C2, C3: footprint Capacitor_SMD:C_1206_3216Metric_Pad1.42x1.75mm_HandSolder -> Capacitor_THT:C_Disc_D5.0mm_W2.5mm_P5.00mm
- R10, R11, R12, R13, R14, R15, R16, R17, R18, R19, R20, R21, R22, R23, R24, R25, R26, R27, R28, R29, R30, R5, R6, R7, R8, R9: footprint Resistor_SMD:R_1206_3216Metric_Pad1.42x1.75mm_HandSolder -> Resistor_THT:R_Axial_DIN0207_L6.3mm_D2.5mm_P7.62mm_Horizontal
Connections:
- net +12V renamed GND
- net GND: no longer C2.1, D1.1 (K), U1.1 (IN)
- new net: C2.1, D1.1 (K), U1.1 (IN)
Other:
- note removed: "Charger battery"
- moved on the sheet: C2, C3, D1, J1, U1

Commit message: pcb desing
Parts:
- added J2: GND, Connector_PinHeader_2.54mm:PinHeader_1x03_P2.54mm_Vertical, symbol Connector:Conn_01x03_Female
Connections:
- net GND1: now also J2.1 (Pin_1); no longer D5.1 (K), D6.1 (K), D7.1 (K), D8.1 (K)
- net GND2: now also J2.2 (Pin_2); no longer D10.1 (K), D11.1 (K), D12.1 (K), D9.1 (K)
- net GND3: now also J2.3 (Pin_3); no longer D13.1 (K), D14.1 (K), D15.1 (K), D16.1 (K)
- net GND4: now also D10.1 (K), D11.1 (K), D12.1 (K), D13.1 (K), D14.1 (K), D15.1 (K), D16.1 (K), D5.1 (K), D6.1 (K), D7.1 (K), D8.1 (K), D9.1 (K)
- net IO16: no longer Q2.2 (B)
- net IO17: no longer Q3.2 (B)
- net IO18: now also Q2.2 (B); no longer Q1.2 (B)
- net IO19: now also Q3.2 (B)
- net IO21: no longer Q4.2 (B)
- net IO22: no longer Q5.2 (B)
- net IO23: now also Q1.2 (B); no longer Q6.2 (B)
- net IO32: now also R26.2
- net IO33: now also Q6.2 (B)
- net IO34: now also Q5.2 (B)
- net IO35: now also Q4.2 (B)
- net IO5: no longer R26.2
Other:
- moved on the sheet: D10, D11, D12, D13, D14, D15, D16, D17, D18, D19, D20, D5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
